Commit message: feat: update morphing_drone URDF mass/inertia and arm length
Co-authored-by: Cursor <cursoragent@cursor.com>

File: assets/urdf/morphing_drone.urdf (robot description, URDF)
Before this commit: robot morphing_drone, 21 links, 20 joints
Links:
- link arm0_link: mass 0.0001 -> 0.1; geometry collision box size=0.12 0.01 0.01; visual box size=0.12 0.01 0.01
- link arm1_link: mass 0.0001 -> 0.1; geometry collision box size=0.12 0.01 0.01; visual box size=0.12 0.01 0.01
- link arm2_link: mass 0.0001 -> 0.1; geometry collision box size=0.12 0.01 0.01; visual box size=0.12 0.01 0.01
- link arm3_link: mass 0.0001 -> 0.1; geometry collision box size=0.12 0.01 0.01; visual box size=0.12 0.01 0.01
- link base_link: mass 0.1 -> 1.4
Joints:
- joint arm0_tilt_joint: origin xyz=0.18 0 0 rpy=0 0 0 -> xyz=0.12 0 0 rpy=0 0 0
- joint arm1_tilt_joint: origin xyz=0.18 0 0 rpy=0 0 0 -> xyz=0.12 0 0 rpy=0 0 0
- joint arm2_tilt_joint: origin xyz=0.18 0 0 rpy=0 0 0 -> xyz=0.12 0 0 rpy=0 0 0
- joint arm3_tilt_joint: origin xyz=0.18 0 0 rpy=0 0 0 -> xyz=0.12 0 0 rpy=0 0 0
